Commit message: [modify] Wheelのprefixのとり方を変更

File: fourth_robot_description/urdf/wheel/wheel.transmission.xacro (robot description, xacro)
@@ -2,10 +2,10 @@
 <robot xmlns:xacro="http://ros.org/wiki/xacro">
   <xacro:macro name="wheel_trans_v0" params="prefix">
-	<transmission name="wheel_${prefix}_trans">
+	<transmission name="${prefix}_wheel_trans">
       <type>transmission_interface/SimpleTransmission</type>
-      <joint name="wheel_${prefix}_joint">
+      <joint name="${prefix}_wheel_joint">
 		<hardwareInterface>VelocityJointInterface</hardwareInterface>
       </joint>
-	  <actuator name="wheel_${prefix}_motor">
+	  <actuator name="${prefix}_wheel_motor">
 		<hardwareInterface>VelocityJointInterface</hardwareInterface>
 		<mechanicalReduction>30</mechanicalReduction>

File: fourth_robot_description/urdf/wheel/wheel.urdf.xacro (robot description, xacro)
@@ -8,11 +8,11 @@
   <property name="wheel_mass" value="2.0"/>
   <xacro:macro name="wheel_v0" params="prefix parent *joint_origin *joint_axis">
-	<joint name="wheel_${prefix}_joint" type="continuous">
+	<joint name="${prefix}_wheel_joint" type="continuous">
 	  <insert_block name="joint_origin"/>
 	  <parent link="${parent}"/>
-	  <child link="wheel_${prefix}_link"/>
+	  <child link="_${prefix}_wheel_link"/>
 	  <insert_block name="joint_axis"/>
 	</joint>
-	<link name="wheel_${prefix}_link">
+	<link name="${prefix}_wheel_link">
 	  <visual>
 		<geometry>
