Commit message: [fix] wheelのtypowを修正

File: fourth_robot_description/urdf/wheel/wheel.gazebo.xacro (robot description, xacro)
@@ -2,5 +2,5 @@
 <robot xmlns:xacro="http://ros.org/wiki/xacro">
   <xacro:macro name="wheel_gazebo_v0" params="prefix">
-	<gazebo reference="wheel_${prefix}_link">
+	<gazebo reference="${prefix}_wheel_link">
 	  <selfCollide>true</selfCollide>
       <mu1 value="0.8" />

File: fourth_robot_description/urdf/wheel/wheel.urdf.xacro (robot description, xacro)
@@ -11,5 +11,5 @@
 	  <insert_block name="joint_origin"/>
 	  <parent link="${parent}"/>
-	  <child link="_${prefix}_wheel_link"/>
+	  <child link="${prefix}_wheel_link"/>
 	  <insert_block name="joint_axis"/>
 	</joint>
