Commit message: [fix] lrfのプラグインをgpu_ray -> ray に変更
これにしないとうまく動きませんでした。

File: fourth_robot_description/urdf/sensors/lrf/lrf.gazebo.xacro (robot description, xacro)
@@ -1,7 +1,7 @@
 <?xml version="1.0"?>
 <robot xmlns:xacro="http://ros.org/wiki/xacro">
-<xacro:macro name="lrf_gazebo_v0" params="prefix min_rad max_rad min_range max_range">
+  <xacro:macro name="lrf_gazebo_v0" params="prefix min_rad max_rad min_range max_range">
 	<gazebo reference="${prefix}_lrf_link">
-      <sensor type="gpu_ray" name="${prefix}_lrf_sensor">
+      <sensor type="ray" name="${prefix}_lrf_sensor">
 		<pose>0 0 0 0 0 0</pose>
 		<visualize>false</visualize>
@@ -27,5 +27,5 @@
           </noise>
 		</ray>
-		<plugin name="gazebo_ros_${prefix}_lrf_controller" filename="libgazebo_ros_gpu_laser.so">
+		<plugin name="gazebo_ros_${prefix}_lrf_controller" filename="libgazebo_ros_laser.so">
           <topicName>/fourth_robot/${prefix}/scan</topicName>
           <frameName>${prefix}_lrf_link</frameName>
