Commit message: [fix] 重心の位置とイナーシャを変更

File: fourth_robot_description/urdf/base/base.urdf.xacro (robot description, xacro)
@@ -20,8 +20,9 @@
 	  </collision>
 	  <inertial>
+		<origin xyz="-0.061 0 -0.002"/>
 		<mass value="45"/>
-		<inertia ixx="1.63567" ixy="0" ixz="-0.47653"
-				 iyy="2.69062" iyz="0"
-				 izz="1.71284" />
+		<inertia ixx="1.64890" ixy="0" ixz="-0.21424"
+				 iyy="2.24766" iyz="0"
+				 izz="1.25664" />
 	  </inertial>
 	</link>

Commit message: Modifying xacros

File: fourth_robot_description/urdf/base/base.urdf.xacro (robot description, xacro)
@@ -4,5 +4,5 @@
   <xacro:macro name="base_v0" params="parent *joint_origin">
 	<joint name="base_link_joint" type="fixed">
-	  <insert_block name="joint_origin"/>
+	  <xacro:insert_block name="joint_origin"/>
 	  <parent link="${parent}"/>
 	  <child link="base_link"/>

File: fourth_robot_description/urdf/sensors/gim30/gim30.urdf.xacro (robot description, xacro)
@@ -4,5 +4,5 @@
   <xacro:macro name="gim30_v0" params="parent *joint_origin">
 	<joint name="gim30_joint" type="fixed">
-      <insert_block name="joint_origin" />
+      <xacro:insert_block name="joint_origin" />
       <parent link="${parent}"/>
       <child link="gim30_link"/>

File: fourth_robot_description/urdf/sensors/gps/gps.urdf.xacro (robot description, xacro)
@@ -4,5 +4,5 @@
   <xacro:macro name="gps_v0" params="parent *joint_origin">
 	<joint name="gps_joint" type="fixed">
-	  <insert_block name="joint_origin"/>
+	  <xacro:insert_block name="joint_origin"/>
 	  <parent link="${parent}"/>
 	  <child link="gps_link"/>

File: fourth_robot_description/urdf/sensors/lrf/lrf.urdf.xacro (robot description, xacro)
@@ -5,5 +5,5 @@
   <xacro:macro name="lrf_v0" params="prefix parent *joint_origin">
 	<joint name="${prefix}_lrf_joint" type="fixed">
-	  <insert_block name="joint_origin"/>
+	  <xacro:insert_block name="joint_origin"/>
 	  <parent link="${parent}"/>
 	  <child link="${prefix}_lrf_link"/>

File: fourth_robot_description/urdf/wheel/wheel.urdf.xacro (robot description, xacro)
@@ -4,13 +4,13 @@
   <xacro:include filename="$(find fourth_robot_description)/urdf/wheel/wheel.transmission.xacro"/>
   <xacro:include filename="$(find fourth_robot_description)/urdf/wheel/wheel.gazebo.xacro"/>
-  <property name="wheel_radius" value="0.0135"/>
-  <property name="wheel_length" value="0.011"/>
-  <property name="wheel_mass" value="0.066"/>
+  <xacro:property name="wheel_radius" value="0.0135"/>
+  <xacro:property name="wheel_length" value="0.011"/>
+  <xacro:property name="wheel_mass" value="0.066"/>
   <xacro:macro name="wheel_v0" params="prefix parent *joint_origin *joint_axis">
 	<joint name="${prefix}_wheel_joint" type="continuous">
-	  <insert_block name="joint_origin"/>
+	  <xacro:insert_block name="joint_origin"/>
 	  <parent link="${parent}"/>
 	  <child link="${prefix}_wheel_link"/>
-	  <insert_block name="joint_axis"/>
+	  <xacro:insert_block name="joint_axis"/>
 	</joint>
 	<link name="${prefix}_wheel_link">
