Commit message: [modify] 全要素にcollisionを追加

File: fourth_robot_description/robots/fourth_robot.urdf.xacro (robot description, xacro)
@@ -30,13 +30,13 @@
   <!-- Gim30 -->
   <xacro:gim30_v0 parent="base_link">
-	<origin xyz="0.12395931 0 0.24578237"/>
+  	<origin xyz="0.12395931 0 0.24578237"/>
   </xacro:gim30_v0>
   <!-- Front LRF -->
   <xacro:lrf_v0 prefix="front" parent="base_link">
-	<origin xyz="0.208 0 -0.0282"/>
+  	<origin xyz="0.208 0 -0.0282"/>
   </xacro:lrf_v0>
   <!-- Rear LRF -->
   <xacro:lrf_v0 prefix="rear" parent="base_link">
-	<origin xyz="-0.452 0 -0.0309" rpy="0 -${M_PI} 0"/>
+  	<origin xyz="-0.452 0 -0.0309" rpy="0 -${M_PI} 0"/>
   </xacro:lrf_v0>
   <!-- ===============  Transmission =============== -->
@@ -44,13 +44,13 @@
   <xacro:wheel_trans_v0 prefix="left"/>
   <!-- =============== Gazebo =============== -->
-    <gazebo>
+  <gazebo>
     <plugin name="gazebo_ros_control" filename="libgazebo_ros_control.so">
       <robotNamespace>/fourth_robot</robotNamespace>
     </plugin>
-	</gazebo>
-	<!-- Base -->
-	<xacro:base_gazebo_v0/>
-	<!-- Wheel -->
-	<xacro:wheel_gazebo_v0 prefix="right"/>
-	<xacro:wheel_gazebo_v0 prefix="left"/>
+  </gazebo>
+  <!-- Base -->
+  <xacro:base_gazebo_v0/>
+  <!-- Wheel -->
+  <xacro:wheel_gazebo_v0 prefix="right"/>
+  <xacro:wheel_gazebo_v0 prefix="left"/>
 </robot>

File: fourth_robot_description/urdf/base/base.urdf.xacro (robot description, xacro)
@@ -14,4 +14,15 @@
 		</geometry>
 	  </visual>
+	  <collision>
+		<geometry>
+		  <mesh filename="package://fourth_robot_description/meshes/STL/base/base_link.stl"/>
+		</geometry>
+	  </collision>
+	  <inertial>
+		<mass value="45"/>
+		<inertia ixx="1.63567" ixy="0" ixz="-0.47653"
+				 iyy="2.69062" iyz="0"
+				 izz="1.71284" />
+	  </inertial>
 	</link>
   </xacro:macro>

File: fourth_robot_description/urdf/common.xacro (robot description, xacro)
@@ -1,4 +1,16 @@
 <?xml version="1.0"?>
-<robot>
+<robot xmlns:xacro="http://ros.org/wiki/xacro">
   <property name="M_PI" value="3.14159274"/>
+  <xacro:macro name="cylinder_inertial" params="mass radius length">
+	<mass value="${mass}"/>
+	<inertia ixx="${((radius*radius)/4 + (length*length)/12)*mass}" ixy="0" ixz="0"
+			 iyy="${((radius*radius)/4 + (length*length)/12)*mass}" iyz="0"
+			 izz="${(mass*radius*radius)/2}" />
+  </xacro:macro>
+  <xacro:macro name="box_inertial" params="mass height width depth">
+	<mass value="${mass}"/>
+	<inertia ixx="${(mass*(width*width+depth*depth))/12}" ixy="0" ixz="0"
+			 iyy="${(mass*(height*height+depth*depth))/12}" iyz="0"
+			 izz="${(mass*(height*height+width*width))/12}" />
+  </xacro:macro>
 </robot>

File: fourth_robot_description/urdf/sensors/gim30/gim30.urdf.xacro (robot description, xacro)
@@ -1,4 +1,5 @@
 <?xml version="1.0"?>
 <robot xmlns:xacro="http://ros.org/wiki/xacro">
+  <xacro:include filename="$(find fourth_robot_description)/urdf/common.xacro"/>
   <xacro:macro name="gim30_v0" params="parent *joint_origin">
 	<joint name="gim30_joint" type="fixed">
@@ -13,4 +14,13 @@
         </geometry>
       </visual>
+	  <collision>
+		<geometry>
+		  <mesh filename="package://fourth_robot_description/meshes/STL/sensors/gim30/gim30.stl"/>
+		</geometry>
+	  </collision>
+	  <inertial>
+		<origin xyz="-0.04 0 -0.1"/>
+		<box_inertial mass="0.85" height="0.1" width="0.05" depth="0.25"/>
+	  </inertial>
     </link>
   </xacro:macro>

File: fourth_robot_description/urdf/sensors/gps/gps.urdf.xacro (robot description, xacro)
@@ -1,4 +1,5 @@
 <?xml version="1.0"?>
 <robot xmlns:xacro="http://ros.org/wiki/xacro">
+  <xacro:include filename="$(find fourth_robot_description)/urdf/common.xacro"/>
   <xacro:macro name="gps_v0" params="parent *joint_origin">
 	<joint name="gps_joint" type="fixed">
@@ -13,4 +14,12 @@
 		</geometry>
 	  </visual>
+	  <collision>
+		<geometry>
+		  <mesh filename="package://fourth_robot_description/meshes/STL/sensors/gps/gps.stl"/>
+		</geometry>
+	  </collision>
+	  <inertial>
+		<cylinder_inertial mass="0.25" radius="0.065" length="0.055"/>
+	  </inertial>
 	</link>
   </xacro:macro>

File: fourth_robot_description/urdf/sensors/lrf/lrf.urdf.xacro (robot description, xacro)
@@ -1,4 +1,5 @@
 <?xml version="1.0"?>
 <robot xmlns:xacro="http://ros.org/wiki/xacro">
+  <xacro:include filename="$(find fourth_robot_description)/urdf/common.xacro"/>
   <xacro:macro name="lrf_v0" params="prefix parent *joint_origin">
 	<joint name="${prefix}_lrf_joint" type="fixed">
@@ -13,4 +14,13 @@
 		</geometry>
 	  </visual>
+	  <collision>
+		<geometry>
+		  <mesh filename="package://fourth_robot_description/meshes/STL/sensors/${prefix}_lrf/${prefix}_lrf.stl"/>
+		</geometry>
+	  </collision>
+	  <inertial>
+		<origin xyz="0 0 -0.0164"/>
+		<box_inertial mass="0.4" height="0.07" width="0.07" depth="0.08"/>
+	  </inertial>
 	</link>
   </xacro:macro>

File: fourth_robot_description/urdf/wheel/wheel.urdf.xacro (robot description, xacro)
@@ -28,8 +28,6 @@
 	  <inertial>
 		<origin xyz="0 -0.003 0" rpy="${-M_PI/2} 0 0"/>
-		<mass value="${wheel_mass}"/>
-		<inertia ixx="${((wheel_radius*wheel_radius)/4 + (wheel_length*wheel_length)/12)*wheel_mass}" ixy="0" ixz="0"
-				 iyy="${((wheel_radius*wheel_radius)/4 + (wheel_length*wheel_length)/12)*wheel_mass}" iyz="0"
-				 izz="${(wheel_mass*wheel_radius*wheel_radius)/2}" />
+		<cylinder_inertial mass="${wheel_mass}"
+						   radius="${wheel_radius}" length="${wheel_length}"/>
 	  </inertial>
 	</link>

Commit message: [fix] front_lrfの位置を修正
高さが間違っていたので修正

File: fourth_robot_description/robots/fourth_robot.urdf.xacro (robot description, xacro)
@@ -34,5 +34,5 @@
   <!-- Front LRF -->
   <xacro:lrf_v0 prefix="front" parent="base_link">
-  	<origin xyz="0.208 0 -0.0282"/>
+  	<origin xyz="0.208 0 -0.025325"/>
   </xacro:lrf_v0>
   <!-- Rear LRF -->

Commit message: [modify] ロボットのnamespaceを決定 wheelの回転方向を修正

File: fourth_robot_description/robots/fourth_robot.urdf.xacro (robot description, xacro)
@@ -21,5 +21,5 @@
   <xacro:wheel_v0 prefix="left" parent="base_link">
 	<origin xyz="0 0.214375 0" rpy="0 0 ${M_PI}"/>
-	<axis xyz="0 1 0"/>
+	<axis xyz="0 -1 0"/>
   </xacro:wheel_v0>
   <!-- Sensors -->
@@ -46,5 +46,5 @@
   <gazebo>
     <plugin name="gazebo_ros_control" filename="libgazebo_ros_control.so">
-      <robotNamespace>/fourth_robot</robotNamespace>
+      <robotNamespace>fourth_robot</robotNamespace>
     </plugin>
   </gazebo>
@@ -54,4 +54,5 @@
   <xacro:wheel_gazebo_v0 prefix="right"/>
   <xacro:wheel_gazebo_v0 prefix="left"/>
+  <xacro:wheel_gazebo_control_v0 rate="25"/>
   <!-- LRF -->
   <xacro:lrf_gazebo_v0 prefix="front"

Commit message: [modify] センサのdescriptionを変更

File: fourth_robot_description/robots/fourth_robot.urdf.xacro (robot description, xacro)
@@ -34,10 +34,22 @@
   <!-- Front LRF -->
   <xacro:lrf_v0 prefix="front" parent="base_link">
-  	<origin xyz="0.208 0 -0.025325"/>
+  	<origin xyz="0.2215 0 -0.02395"/>
   </xacro:lrf_v0>
   <!-- Rear LRF -->
   <xacro:lrf_v0 prefix="rear" parent="base_link">
-  	<origin xyz="-0.452 0 -0.0309" rpy="0 -${M_PI} 0"/>
+  	<origin xyz="-0.452 0 -0.04025" rpy="0 -${M_PI} 0"/>
   </xacro:lrf_v0>
+  <link name="lrf_link"/>
+  <joint name="lrf_link_joint" type="fixed">
+	<parent link="base_link"/>
+	<child link="lrf_link"/>
+	<origin xyz="0 0 -0.0321"/>
+  </joint>
+  <link name="imu_link"/>
+  <joint name="imu_link_joint" type="fixed">
+	<parent link="base_link"/>
+	<child link="imu_link"/>
+	<origin xyz="0 0 0.051"/>
+  </joint>
   <!-- ===============  Transmission =============== -->
   <xacro:wheel_trans_v0 prefix="right"/>

Commit message: [modify] gazeboモデルの名前空間を削除

File: fourth_robot_description/robots/fourth_robot.urdf.xacro (robot description, xacro)
@@ -50,5 +50,5 @@
 	<parent link="base_link"/>
 	<child link="imu_link"/>
-	<origin xyz="0 0 0.051"/>
+	<origin xyz="0 0 0.051" rpy="0 0 0" />
   </joint>
   <!-- ===============  Transmission =============== -->
@@ -58,5 +58,5 @@
   <gazebo>
     <plugin name="gazebo_ros_control" filename="libgazebo_ros_control.so">
-      <robotNamespace>fourth_robot</robotNamespace>
+      <!-- <robotNamespace>fourth_robot</robotNamespace> -->
     </plugin>
   </gazebo>
@@ -69,8 +69,8 @@
   <!-- LRF -->
   <xacro:lrf_gazebo_v0 prefix="front"
-					   min_rad="-${M_PI/2}" max_rad="${M_PI/2}"
-					   min_range="0.10" max_range="10.0"/>
+					   min_rad="-1.65806278939" max_rad="-1.65806278939"
+					   min_range="0.10" max_range="60.0"/>
   <xacro:lrf_gazebo_v0 prefix="rear"
-					   min_rad="-${110*M_PI/180}" max_rad="${110*M_PI/180}"
-					   min_range="0.10" max_range="5.0"/>
+					   min_rad="-2.35619449019" max_rad="2.35619449019"
+					   min_range="0.10" max_range="60.0"/>
 </robot>

File: fourth_robot_description/urdf/base/base.gazebo.xacro (robot description, xacro)
@@ -3,5 +3,5 @@
   <xacro:macro name="base_gazebo_v0">
 	<gazebo reference="base_link">
-	  <selfCollide>true</selfCollide>
+	  <selfCollide>false</selfCollide>
       <mu1 value="0.05" />
       <mu2 value="0.05" />

File: fourth_robot_description/urdf/sensors/lrf/lrf.gazebo.xacro (robot description, xacro)
@@ -5,5 +5,5 @@
       <sensor type="ray" name="${prefix}_lrf_sensor">
 		<pose>0 0 0 0 0 0</pose>
-		<visualize>false</visualize>
+		<visualize>true</visualize>
 		<update_rate>40</update_rate>
 		<ray>
@@ -28,5 +28,5 @@
 		</ray>
 		<plugin name="gazebo_ros_${prefix}_lrf_controller" filename="libgazebo_ros_laser.so">
-          <topicName>/fourth_robot/${prefix}/scan</topicName>
+          <topicName>${prefix}/scan</topicName>
           <frameName>${prefix}_lrf_link</frameName>
 		</plugin>

File: fourth_robot_description/urdf/wheel/wheel.gazebo.xacro (robot description, xacro)
@@ -3,5 +3,5 @@
   <xacro:macro name="wheel_gazebo_v0" params="prefix">
 	<gazebo reference="${prefix}_wheel_link">
-	  <selfCollide>true</selfCollide>
+	  <selfCollide>false</selfCollide>
       <mu1 value="0.8" />
       <mu2 value="0.8" />

Commit message: [modify] kinematics about sensors

File: fourth_robot_description/robots/fourth_robot.urdf.xacro (robot description, xacro)
@@ -30,13 +30,13 @@
   <!-- Gim30 -->
   <xacro:gim30_v0 parent="base_link">
-  	<origin xyz="0.12395931 0 0.24578237"/>
+  	<origin xyz="0.07395931 0 0.24578237"/>
   </xacro:gim30_v0>
   <!-- Front LRF -->
   <xacro:lrf_v0 prefix="front" parent="base_link">
-  	<origin xyz="0.2215 0 -0.02395"/>
+  	<origin xyz="0.2215 0 0.04684"/>
   </xacro:lrf_v0>
   <!-- Rear LRF -->
   <xacro:lrf_v0 prefix="rear" parent="base_link">
-  	<origin xyz="-0.452 0 -0.04025" rpy="0 -${M_PI} 0"/>
+  	<origin xyz="-0.452 0 0.04684" rpy="0 0 -${M_PI}"/>
   </xacro:lrf_v0>
   <link name="lrf_link"/>
@@ -44,5 +44,5 @@
 	<parent link="base_link"/>
 	<child link="lrf_link"/>
-	<origin xyz="0 0 -0.0321"/>
+	<origin xyz="0 0 0.04684"/>
   </joint>
   <link name="imu_link"/>
@@ -66,5 +66,5 @@
   <xacro:wheel_gazebo_v0 prefix="right"/>
   <xacro:wheel_gazebo_v0 prefix="left"/>
-  <xacro:wheel_gazebo_control_v0 rate="25"/>
+  <!-- <xacro:wheel_gazebo_control_v0 rate="25"/> -->
   <!-- LRF -->
   <xacro:lrf_gazebo_v0 prefix="front"

Commit message: Made architect2

File: fourth_robot_description/robots/fourth_robot.urdf.xacro (robot description, xacro)
@@ -15,27 +15,27 @@
   <!-- Right Wheel -->
   <xacro:wheel_v0 prefix="right" parent="base_link">
-	<origin xyz="0 -0.214375 0"/>
-	<axis xyz="0 1 0"/>
+        <origin xyz="-0.014 -0.0695 0.0115" rpy="0 0 0"/>
+        <axis xyz="0 1 0"/>
   </xacro:wheel_v0>
   <!-- Left Wheel -->
   <xacro:wheel_v0 prefix="left" parent="base_link">
-	<origin xyz="0 0.214375 0" rpy="0 0 ${M_PI}"/>
-	<axis xyz="0 -1 0"/>
+        <origin xyz="-0.014 0.0695 0.0115" rpy="0 0 ${M_PI}"/>
+        <axis xyz="0 -1 0"/>
   </xacro:wheel_v0>
   <!-- Sensors -->
   <!-- GPS -->
-  <xacro:gps_v0 parent="base_link">
+ <!-- <xacro:gps_v0 parent="base_link">
 	<origin xyz="-0.06229 0 0.420552" rpy="0 0 -${M_PI}"/>
-  </xacro:gps_v0>
+  </xacro:gps_v0>-->
   <!-- Gim30 -->
-  <xacro:gim30_v0 parent="base_link">
+  <!--<xacro:gim30_v0 parent="base_link">
   	<origin xyz="0.07395931 0 0.24578237"/>
-  </xacro:gim30_v0>
+  </xacro:gim30_v0>-->
   <!-- Front LRF -->
-  <xacro:lrf_v0 prefix="front" parent="base_link">
+<!--  <xacro:lrf_v0 prefix="front" parent="base_link">
   	<origin xyz="0.2215 0 0.04684"/>
-  </xacro:lrf_v0>
+  </xacro:lrf_v0>-->
   <!-- Rear LRF -->
-  <xacro:lrf_v0 prefix="rear" parent="base_link">
+<!--  <xacro:lrf_v0 prefix="rear" parent="base_link">
   	<origin xyz="-0.452 0 0.04684" rpy="0 0 -${M_PI}"/>
   </xacro:lrf_v0>
@@ -45,5 +45,5 @@
 	<child link="lrf_link"/>
 	<origin xyz="0 0 0.04684"/>
-  </joint>
+  </joint>-->
   <link name="imu_link"/>
   <joint name="imu_link_joint" type="fixed">
@@ -68,9 +68,9 @@
   <!-- <xacro:wheel_gazebo_control_v0 rate="25"/> -->
   <!-- LRF -->
-  <xacro:lrf_gazebo_v0 prefix="front"
+  <!--<xacro:lrf_gazebo_v0 prefix="front"
 					   min_rad="-1.65806278939" max_rad="1.65806278939"
 					   min_range="0.10" max_range="60.0"/>
   <xacro:lrf_gazebo_v0 prefix="rear"
 					   min_rad="-2.35619449019" max_rad="2.35619449019"
-					   min_range="0.10" max_range="60.0"/>
+                                           min_range="0.10" max_range="60.0"/>-->
 </robot>

File: fourth_robot_description/urdf/base/base.urdf.xacro (robot description, xacro)
@@ -10,19 +10,22 @@
 	<link name="base_link">
 	  <visual>
+                <origin xyz="0 0 0" rpy="0 0 0" />
 		<geometry>
-		  <mesh filename="package://fourth_robot_description/meshes/DAE/base/base_link.dae"/>
+                  <!--<mesh filename="package://fourth_robot_description/meshes/DAE/base/base_link.dae"/>-->
+                  <mesh filename="package://fourth_robot_description/meshes/STL/base/Architect_assem_appearance.stl"/>
 		</geometry>
 	  </visual>
 	  <collision>
 		<geometry>
-		  <mesh filename="package://fourth_robot_description/meshes/STL/base/base_link.stl"/>
+                  <!--<mesh filename="package://fourth_robot_description/meshes/STL/base/base_link.stl"/>-->
+                  <mesh filename="package://fourth_robot_description/meshes/STL/base/Architect_assem_collision.stl"/>
 		</geometry>
 	  </collision>
 	  <inertial>
-		<origin xyz="-0.061 0 -0.002"/>
-		<mass value="45"/>
-		<inertia ixx="1.64890" ixy="0" ixz="-0.21424"
-				 iyy="2.24766" iyz="0"
-				 izz="1.25664" />
+                <origin xyz="0 0 0"/>
+                <mass value="2.4"/>
+                <inertia ixx="0.0008255" ixy="0" ixz="0.00001601"
+                                 iyy="0.0007067" iyz="-0.0000000009905"
+                                 izz="0.0004498" />
 	  </inertial>
 	</link>

File: fourth_robot_description/urdf/wheel/wheel.urdf.xacro (robot description, xacro)
@@ -4,7 +4,7 @@
   <xacro:include filename="$(find fourth_robot_description)/urdf/wheel/wheel.transmission.xacro"/>
   <xacro:include filename="$(find fourth_robot_description)/urdf/wheel/wheel.gazebo.xacro"/>
-  <property name="wheel_radius" value="0.20316"/>
-  <property name="wheel_length" value="0.032"/>
-  <property name="wheel_mass" value="2.0"/>
+  <property name="wheel_radius" value="0.0135"/>
+  <property name="wheel_length" value="0.011"/>
+  <property name="wheel_mass" value="0.066"/>
   <xacro:macro name="wheel_v0" params="prefix parent *joint_origin *joint_axis">
 	<joint name="${prefix}_wheel_joint" type="continuous">
@@ -15,11 +15,13 @@
 	</joint>
 	<link name="${prefix}_wheel_link">
-	  <visual>
+          <visual>
+          <origin xyz="0 0 0" rpy="${-M_PI/2} 0 0"/>
 		<geometry>
-		  <mesh filename="package://fourth_robot_description/meshes/DAE/wheel/wheel_link.dae"/>
+                  <!--<mesh filename="package://fourth_robot_description/meshes/DAE/wheel/wheel_link.dae"/>-->
+                  <cylinder radius="${wheel_radius}" length="${wheel_length}"/>
 		</geometry>
 	  </visual>
 	  <collision>
-		<origin xyz="0 -0.003 0" rpy="${-M_PI/2} 0 0"/>
+                <origin xyz="0 0 0" rpy="${-M_PI/2} 0 0"/>
 		<geometry>
 		  <cylinder radius="${wheel_radius}" length="${wheel_length}"/>

Commit message: Added stereo camera

File: fourth_robot_description/robots/fourth_robot.urdf.xacro (robot description, xacro)
@@ -6,4 +6,5 @@
   <xacro:include filename="$(find fourth_robot_description)/urdf/sensors/gim30/gim30.urdf.xacro"/>
   <xacro:include filename="$(find fourth_robot_description)/urdf/sensors/lrf/lrf.urdf.xacro"/>
+  <xacro:include filename="$(find fourth_robot_description)/urdf/sensors/stereo_camera/stereo_camera.urdf.xacro"/>
   <!-- =============== Link & Joint =============== -->
   <!-- Base -->
@@ -46,4 +47,8 @@
 	<origin xyz="0 0 0.04684"/>
   </joint>-->
+  <!--stereo camera-->
+  <xacro:stereo_camera prefix="upper" parent="base_link">
+    <origin xyz="0 0 0.2" rpy="0 0 0"/>
+  </xacro:stereo_camera>
   <link name="imu_link"/>
   <joint name="imu_link_joint" type="fixed">
@@ -74,3 +79,5 @@
 					   min_rad="-2.35619449019" max_rad="2.35619449019"
                                            min_range="0.10" max_range="60.0"/>-->
+  <!--Stereo Camera-->
+  <xacro:stereo_camera_gazebo prefix="upper"/>
 </robot>

Commit message: Change collision

File: fourth_robot_description/robots/fourth_robot.urdf.xacro (robot description, xacro)
@@ -3,4 +3,5 @@
   <xacro:include filename="$(find fourth_robot_description)/urdf/base/base.urdf.xacro"/>
   <xacro:include filename="$(find fourth_robot_description)/urdf/wheel/wheel.urdf.xacro"/>
+  <xacro:include filename="$(find fourth_robot_description)/urdf/wheel/follow_wheel.urdf.xacro"/>
 <!--  <xacro:include filename="$(find fourth_robot_description)/urdf/sensors/gps/gps.urdf.xacro"/>
   <xacro:include filename="$(find fourth_robot_description)/urdf/sensors/gim30/gim30.urdf.xacro"/>
@@ -24,4 +25,9 @@
         <axis xyz="0 -1 0"/>
   </xacro:wheel_v0>
+  <!-- Front Wheel -->
+  <xacro:follow_wheel_v0 prefix="front" parent="base_link">
+        <origin xyz="0.05 0 0.0115" rpy="0 0 ${M_PI}"/>
+        <axis xyz="0 -1 0"/>
+  </xacro:follow_wheel_v0>
   <!-- Sensors -->
   <!-- GPS -->
@@ -71,4 +77,5 @@
   <xacro:wheel_gazebo_v0 prefix="right"/>
   <xacro:wheel_gazebo_v0 prefix="left"/>
+  <xacro:follow_wheel_gazebo_v0 prefix="front"/>
   <!-- <xacro:wheel_gazebo_control_v0 rate="25"/> -->
   <!-- LRF -->

Commit message: Modified camera

File: fourth_robot_description/robots/fourth_robot.urdf.xacro (robot description, xacro)
@@ -55,5 +55,5 @@
   <!--stereo camera-->
   <xacro:stereo_camera prefix="upper" parent="base_link">
-    <origin xyz="0 0 0.2" rpy="0 0 0"/>
+    <origin xyz="0 0 0.16" rpy="0 0.31 0"/>
   </xacro:stereo_camera>
   <link name="imu_link"/>

File: fourth_robot_description/urdf/sensors/stereo_camera/stereo_camera.gazebo.xacro (robot description, xacro)
@@ -6,8 +6,8 @@
       <update_rate>30.0</update_rate>
       <camera name="left">
-        <horizontal_fov>1.3962634</horizontal_fov>
+        <horizontal_fov>2.2</horizontal_fov>
         <image>
-          <width>800</width>
-          <height>800</height>
+          <width>752</width>
+          <height>480</height>
           <format>R8G8B8</format>
         </image>
@@ -24,8 +24,8 @@
       <camera name="right">
         <pose>0 -0.07 0 0 0 0</pose>
-        <horizontal_fov>1.3962634</horizontal_fov>
+        <horizontal_fov>2.2</horizontal_fov>
         <image>
-          <width>800</width>
-          <height>800</height>
+          <width>752</width>
+          <height>480</height>
           <format>R8G8B8</format>
         </image>

File: fourth_robot_description/urdf/sensors/stereo_camera/stereo_camera.urdf.xacro (robot description, xacro)
@@ -12,5 +12,5 @@
             <origin xyz="0 0 0" rpy="0 0 0"/>
             <geometry>
-              <box size="0.05 0.05 0.05"/>
+              <box size="0.01 0.01 0.01"/>
             </geometry>
           </collision>
@@ -18,5 +18,5 @@
             <origin xyz="0 0 0" rpy="0 0 0"/>
             <geometry>
-              <box size="0.05 0.05 0.05"/>
+              <box size="0.01 0.01 0.01"/>
             </geometry>
             <material name="red"/>
