Commit message: Delete6

File: architect_description/urdf/base/base.urdf.xacro (robot description, xacro)
@@ -12,5 +12,4 @@
                 <origin xyz="0 0 0" rpy="0 0 0" />
 		<geometry>
-                  <!--<mesh filename="package://architect_description/meshes/DAE/base/base_link.dae"/>-->
                   <mesh filename="package://architect_description/meshes/STL/base/Architect_assem_appearance.stl"/>
 		</geometry>
@@ -18,5 +17,4 @@
 	  <collision>
 		<geometry>
-                  <!--<mesh filename="package://architect_description/meshes/STL/base/base_link.stl"/>-->
                   <mesh filename="package://architect_description/meshes/STL/base/Architect_assem_collision.stl"/>
 		</geometry>
